File: fifo-p3f/FIFO_P.kicad_pcb (KiCad board)
At the start: 4 copper layers, 100 x 66.5 mm, 99 parts, among them J1 Vin, J2 Jack-DC, J3 Screw_Terminal_01x08, J4 XWCLK, J5 XRCLK, J6 Conn_02x04_Odd_Even, J7 Start Trigger, J8 Vout, Q1 DMP3099L, SW1 Rotary_Encoder_61C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

Commit message: Added assembly instructions, removed TeX logs, and reorganized docs
Parts:
- removed C36: 0u1, Capacitor_SMD:C_0805_2012Metric_Pad1.15x1.40mm_HandSolder
- added C47: 1n, Capacitor_SMD:C_0805_2012Metric_Pad1.15x1.40mm_HandSolder, B.Cu at (114.5, 73.0)
- added R17: 5k1, Resistor_SMD:R_0805_2012Metric_Pad1.15x1.40mm_HandSolder, B.Cu at (95.5, 78.3)
- added R18: 5k1, Resistor_SMD:R_0805_2012Metric_Pad1.15x1.40mm_HandSolder, B.Cu at (97.8, 78.3)
- added R19: 49R9, Resistor_SMD:R_0805_2012Metric_Pad1.15x1.40mm_HandSolder, B.Cu at (114.5, 78.2)
- added R20: 22R, Resistor_SMD:R_0805_2012Metric_Pad1.15x1.40mm_HandSolder, B.Cu at (120.5, 78.2)
- R12: value 1k1 -> 4k3
- R14: value 4k3 -> 1k1
- RV2: value 1k -> 10k
Connections:
- R12 pad 1: +5V -> Net-(R12-Pad1)
- R16 pad 1: PROG_ADC -> Net-(C47-Pad1)
- R8 pad 1: Net-(R8-Pad1) -> Net-(R12-Pad1)
- U14 pad 2: Net-(R8-Pad1) -> Net-(R12-Pad1)
- U16 pad 1: PROG_ADC -> Net-(C47-Pad1)
- U16 pad 5: Net-(R8-Pad1) -> Net-(R17-Pad1)
Routing:
- net PROG_ADC: track 29.3 -> 15.3 mm
- net Net-(R12-Pad1): track 0.00 -> 10.9 mm, vias 0 -> 1
- net Net-(R8-Pad1): track 10.7 -> 0.00 mm
- net Net-(R17-Pad1): track 0.00 -> 10.6 mm
- net Net-(C47-Pad1): track 0.00 -> 8.78 mm
- net Net-(R19-Pad1): track 0.00 -> 4.44 mm
- net GND: track 204.9 -> 209.0 mm
- net Net-(RV2-Pad1): track 9.96 -> 6.47 mm
- net Net-(C47-Pad2): track 5.61 -> 9.07 mm, vias 1 -> 2
- net +5V: track 203.1 -> 206.3 mm
